File: ProspectBoards.kicad_pcb (KiCad board)
At the start: 2 copper layers, 100.1 x 99.7 mm, 45 parts, among them J1 Conn_01x02_Female, J2 JTAG, J3 USB_B_Mini, J4 Conn_01x02_Female, J5 Conn_01x02_Female, SW1 SW_SPST, SW6 SW_SPDT, U1 LTC4054, U2 ESP32-S2-WROVER, U3 CH330N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

Commit message: Gerbers
Gerbers for Order
Other:
- board size 100.1 x 99.7 mm -> 100 x 99.7 mm
- net class Default removed
