File: CAD/ProspectBoards.kicad_sch (KiCad schematic)
At the start: 36 parts, among them J1 Conn_01x02_Female, J2 JTAG, J3 USB_B_Mini, J4 Conn_01x02_Female, J5 Conn_01x02_Female, SW1 SW_SPST, SW6 SW_SPDT, U1 LTC4054, U2 ESP32-S2-WROVER, U3 CH330N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

Commit message: Footprint Fixes
FootPrint fix for the Stupid Ass Button that suxs
Parts:
- SW1, SW_Reset1: footprint BadgePirate:Switch_Tactile_SMD_B3U-1000P-BPVersion -> BadgePirates:Switch_Tactile_SMD_B3U-1000P-BPVersion
Changed lines of the file:
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@@
     (property "Reference" "SW_Reset1" (id 0) (at 31.75 119.761 0))
     (property "Value" "Reset_Btn" (id 1) (at 31.75 122.0724 0))
-    (property "Footprint" "BadgePirate:Switch_Tactile_SMD_B3U-1000P-BPVersion" (id 2) (at 31.75 121.92 0)
+    (property "Footprint" "BadgePirates:Switch_Tactile_SMD_B3U-1000P-BPVersion" (id 2) (at 31.75 121.92 0)
       (effects (font (size 1.27 1.27)) hide)
     )
@@
     (property "Reference" "SW1" (id 0) (at 88.9 16.891 0))
     (property "Value" "SW_SPST" (id 1) (at 88.9 19.2024 0))
-    (property "Footprint" "BadgePirate:Switch_Tactile_SMD_B3U-1000P-BPVersion" (id 2) (at 88.9 22.86 0)
+    (property "Footprint" "BadgePirates:Switch_Tactile_SMD_B3U-1000P-BPVersion" (id 2) (at 88.9 22.86 0)
       (effects (font (size 1.27 1.27)) hide)
     )
@@
     )
     (path "/00000000-0000-0000-0000-000061ceeaab"
-      (reference "SW1") (unit 1) (value "SW_SPST") (footprint "BadgePirate:Switch_Tactile_SMD_B3U-1000P-BPVersion")
+      (reference "SW1") (unit 1) (value "SW_SPST") (footprint "BadgePirates:Switch_Tactile_SMD_B3U-1000P-BPVersion")
     )
     (path "/00000000-0000-0000-0000-0000614a1475"
@@
     )
     (path "/00000000-0000-0000-0000-0000615b1b47"
-      (reference "SW_Reset1") (unit 1) (value "Reset_Btn") (footprint "BadgePirate:Switch_Tactile_SMD_B3U-1000P-BPVersion")
+      (reference "SW_Reset1") (unit 1) (value "Reset_Btn") (footprint "BadgePirates:Switch_Tactile_SMD_B3U-1000P-BPVersion")
     )
     (path "/00000000-0000-0000-0000-0000616a16bf"
